Commit message: Franka Panda picking demo

File: examples/applications/non_stop_picking/resources/panda/panda.urdf (robot description, URDF)
Before this commit: robot panda, 12 links, 11 joints
Links:
- link panda_link5: geometry collision mesh filename=package://franka_description/meshes/link5_collision.STL; visual mesh filename=file:///home/yiming/link5.dae

Commit message: Multi threaded non-stop-picking

File: examples/applications/non_stop_picking/resources/panda/panda.urdf (robot description, URDF)
Before this commit: robot panda, 12 links, 11 joints
Links:
- link panda_leftfinger: geometry collision mesh filename=package://franka_description/meshes/leftfinger_collision.STL; visual mesh filename=package://franka_description_dae/meshes/leftfinger.dae
- link panda_link5: geometry collision mesh filename=package://franka_description/meshes/link5_collision.STL; visual mesh filename=package://franka_description_dae/meshes/link5.dae
- link panda_link6: geometry collision mesh filename=package://franka_description/meshes/link6_collision.STL; visual mesh filename=package://franka_description_dae/meshes/link6.dae
- link panda_link7: geometry collision mesh filename=package://franka_description/meshes/link7_collision.STL; visual mesh filename=package://franka_description_dae/meshes/link7.dae
- link panda_rightfinger: geometry collision mesh filename=package://franka_description/meshes/rightfinger_collision.S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; visual mesh filename=package://franka_description_dae/meshes/rightfinger.dae

Commit message: add franka box picking demo

File: examples/applications/non_stop_picking/resources/panda/panda.urdf (robot description, URDF)
Before this commit: robot panda, 12 links, 11 joints
Links:
- link panda_hand: geometry collision mesh filename=package://franka_description/meshes/hand_collision.STL; visual mesh filename=package://franka_description/meshes/hand.dae
- link panda_leftfinger: geometry collision mesh filename=package://franka_description/meshes/leftfinger_collision.STL; visual mesh filename=package://franka_description/meshes/leftfinger.dae
- link panda_link0: geometry collision mesh filename=package://franka_description/meshes/link0_collision.STL; visual mesh filename=package://franka_description/meshes/link0.dae
- link panda_link1: geometry collision mesh filename=package://franka_description/meshes/link1_collision.STL; visual mesh filename=package://franka_description/meshes/link1.dae
- link panda_link2: geometry collision mesh filename=package://franka_description/meshes/link2_collision.STL; visual mesh filename=package://franka_description/meshes/link2.dae
- link panda_link3: geometry collision mesh filename=package://franka_description/meshes/link3_collision.STL; visual mesh filename=package://franka_description/meshes/link3.dae
- link panda_link4: geometry collision mesh filename=package://franka_description/meshes/link4_collision.STL; visual mesh filename=package://franka_description/meshes/link4.dae
- link panda_link5: geometry collision mesh filename=package://franka_description/meshes/link5_collision.STL; visual mesh filename=package://franka_description/meshes/link5.dae
- link panda_link6: geometry collision mesh filename=package://franka_description/meshes/link6_collision.STL; visual mesh filename=package://franka_description/meshes/link6.dae
- link panda_link7: geometry collision mesh filename=package://franka_description/meshes/link7_collision.STL; visual mesh filename=package://franka_description/meshes/link7.dae
- link panda_rightfinger: geometry collision mesh filename=package://franka_description/meshes/rightfinger_collision.S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; visual mesh filename=package://franka_description/meshes/rightfinger.dae
